File: Breakout_Board.brd (EAGLE design)
At the start: 100 x 80 mm, 97 parts, among them IC1 RH-0505S/H6, IC103 ADE7880, IC105 7805TV, Q101 16M384, U101 ADR512ARTZ-REEL7, U102 SI8640BD-B-IS, U103 SI8641BD-B-IS, X1 231-538/001-000, X101 STL266-04, X103 MKDSN1,5/2-5,08

Commit message: -updated sch and brd, added pdf files
Parts:
- removed C1: 1uF, rcl:C0603K
- removed C132: 47u, rcl:PANASONIC_D
- removed C2, C5: 2n2, rcl:C0603K
- removed IC105: 7805TV, linear:TO220V
- removed R1, R15, R18, R6, R7: 2R7, rcl:R0805
- removed R17, R3, R4, R8, R9: 150R, rcl:R0805
- removed R20, R21, R22, R23, R24, R25: 1k, rcl:R0603
- removed X1: 231-538/001-000, con-wago_5.08mm:P-231-538/001-000
- added C109: 2n2, rcl:C0603K
- added C118: 10u, rcl:PANASONIC_B
- added C122, C124: 100n, rcl:C0603K
- added IC101: ADE7880, AnalogDevices_own:BREAKOUT40P
- added R104, R105, R106: 162k, rcl:R0805
- added R125, R136: 196k, rcl:R0805
- added R137, R138, R139: 1k, rcl:R0805
- added R140, R141, R142: 1k, rcl:R0603
- added R143: 2k1, rcl:R0603
- added R145, R146, R147, R148, R149, R150, R151, R152: 10k, rcl:R0603
- added X102: STL266-04, con-riacon:7.62MM-4POL
- C101, C104: value 30pF -> 2n2
- C112: value 2n2 -> 220n
- C113: value 220n -> 4u7; device rcl:C0603K -> rcl:PANASONIC_B
- C114, C116: value 4u7 -> 30pF; device rcl:PANASONIC_B -> rcl:C0603K
- C117: value (none) -> 4u7; device rcl:C0603K -> rcl:PANASONIC_B
- C119: value 10u -> 100n; device rcl:PANASONIC_B -> rcl:C0603K
- C120, C125, C129: value (none) -> 100n
- C121: value (none) -> 1uF
- C127, C131: value 100n -> 47u; device rcl:C0603K -> rcl:PANASONIC_D
- C128: value 47u -> 100n; device rcl:PANASONIC_D -> rcl:C0603K
- IC103: value ADE7880 -> 7805TV; device AnalogDevices_own:BREAKOUT40P -> linear:TO220V
- R107, R108, R109: value 162k -> 2R7
- R113, R114: value 196k -> 2R7
- R115, R116, R117, R118: value 196k -> 150R
- R122: value 1k -> 150R
- R123, R124: value 1k -> 196k
- R131: value 2k1 -> 1k
- R132, R133: value 10k -> 1k
- R134, R135: value 10k -> 196k; device rcl:R0603 -> rcl:R0805
- X101: value STL266-04 -> 231-538/001-000; device con-riacon:7.62MM-4POL -> con-wago_5.08mm:P-231-538/001-000
- moved R135 74.2 mm to (30.5, 20.1)
- moved R134 65.3 mm to (30.5, 12.4)
- moved R107 62.0 mm to (10.4, 73.7), turned to 90 degrees
- moved R116 59.9 mm to (10.4, 68.8), turned to 90 degrees
- moved IC103 57.9 mm to (100.1, 54.1)
- moved C101 56.8 mm to (17.8, 72.1), turned to 180 degrees
- moved R133 56.3 mm to (17.8, 37.1)
- moved R128 55.3 mm to (17.8, 64.8), turned to 0 degrees
- moved C104 55.2 mm to (17.8, 60.2), turned to 0 degrees
- moved R108 49.2 mm to (14.0, 68.8), turned to 90 degrees
- moved R129 48.7 mm to (17.8, 57.9), turned to 0 degrees
- moved R117 48.1 mm to (10.4, 63.8), turned to 90 degrees
- moved R115 47.4 mm to (14.0, 73.7), turned to 90 degrees
- moved C121 44.1 mm to (51.1, 31.8), turned to 0 degrees
- moved R130 41.0 mm to (17.8, 54.6), turned to 0 degrees
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- renumbered C3 to C102, C4 to C103, C6 to C105, C7 to C106, C8 to C107, C9 to C108, IC1 to IC102, R10 to R110, R11 to R111, R12 to R119, R13 to R120, R14 to R112, R16 to R121, R19 to R127, R2 to R126, R5 to R144
Connections:
- removed net N$42: R133.2, U103.10
- new net N$16: R150.2, U103.10
- net !SS: now also IC101.39, R149.1; no longer IC103.39
- net AVDD: now also C112.1, C113.+, IC101.24; no longer C113.1, C114.+, IC103.24
- net DVDD: now also C117.+, IC101.5; no longer C116.+, IC103.5
- net GND: now also C112.2, C113.-, C114.2, C116.1, C117.-, C118.-, C119.2, C122.2, C124.2, C125.1, IC101.25, IC101.3, IC101.6, R107.1, R108.2, R109.1, R113.1, R114.2, R115.1, R116.2, R117.1, R118.2, R122.2; no longer C1.2, C113.2, C114.-, C116.-, C117.2, C119.-, C125.2, C126.1, C2.2, C5.1, IC103.25, IC103.3, IC103.6, R1.1, R15.1, R17.2, R18.2, R3.1, R4.2, R6.2, R7.1, R8.1, R9.2
- net GND_P: now also C126.1, C127.-, C128.2, C131.-, IC103.2; no longer C127.1, C128.-, C131.2, C132.-, IC105.2
- net IAN: now also IC101.8; no longer IC103.8
- net IAP: now also C101.1, IC101.7; no longer C2.1, IC103.7
- net IBN: now also C104.2, IC101.12, R129.2; no longer C5.2, IC103.12, R21.2
- net IBP: now also IC101.9, R128.2; no longer IC103.9, R20.2
- net ICN: now also IC101.14, R131.2; no longer IC103.14, R23.2
- net ICP: now also IC101.13, R130.2; no longer IC103.13, R22.2
- net INH: now also R113.2, R132.1, X101.L7; no longer R15.2, R24.1, X1.L7
- net INL: now also R114.1, R122.1, R133.1, X101.L8; no longer R17.1, R18.1, R25.1, X1.L8
- net INN: now also IC101.16, R133.2; no longer IC103.16, R25.2
- net INP: now also IC101.15, R132.2; no longer IC103.15, R24.2
- net L1H: now also R107.2, R115.2, X101.L1; no longer R1.2, R3.2, X1.L1
- net L1L: now also R108.1, R116.1, X101.L2; no longer R4.1, R6.1, X1.L2
- net L2H: now also R109.2, R117.2, R128.1, X101.L3; no longer R20.1, R7.2, R8.2, X1.L3
- net L2L: now also R118.1, R129.1, X101.L4; no longer R21.1, R9.1, X1.L4
- net L3H: now also R130.1, X101.L5; no longer R22.1, X1.L5
- net L3L: now also R131.1, X101.L6; no longer R23.1, X1.L6
- net MISO: now also IC101.37, R147.1; no longer IC103.37
- net MOSI: now also IC101.38, R148.1; no longer IC103.38
- net N$1: now also R104.1; no longer R107.1
- net N$10: now also X102.P$3; no longer X101.P$3
- net N$11: now also R106.1; no longer R109.1
- net N$12: now also R106.2, R125.1; no longer R109.2, R115.1
- net N$13: now also R125.2, R136.1; no longer R115.2, R118.1
- net N$14: now also R136.2, R139.2, R142.1; no longer R118.2, R124.2, R130.1
- net N$15: now also X102.P$2; no longer X101.P$2
- net N$2: now also R104.2, R123.1; no longer R107.2, R113.1
- net N$25: now also IC101.2, R145.1; no longer IC103.2, R132.1
- net N$3: now also R123.2, R134.1; no longer R113.2, R116.1
- net N$30: now also IC101.4; no longer IC103.4
- net N$35: now also IC101.33; no longer IC103.33
- net N$36: now also IC101.34; no longer IC103.34
- net N$37: now also IC101.35; no longer IC103.35
- net N$38: now also IC101.29; no longer IC103.29
- net N$39: now also IC101.32; no longer IC103.32
- net N$4: now also R134.2, R137.2, R140.1; no longer R116.2, R122.2, R128.1
- net N$40: now also R152.1; no longer R135.1
- net N$41: now also R151.1; no longer R134.1
- net N$46: now also C130.1, C131.+, IC103.1; no longer C131.1, C132.+, IC105.1
- net N$5: now also X102.P$4; no longer X101.P$4
- net N$6: now also R105.1; no longer R108.1
- net N$7: now also R105.2, R124.1; no longer R108.2, R114.1
- net N$8: now also R124.2, R135.1; no longer R114.2, R117.1
- net N$9: now also R135.2, R138.2, R141.1; no longer R117.2, R123.2, R129.1
- net REF: now also C119.1, C121.1, IC101.17, R143.1; no longer C1.1, C117.1, IC103.17, R131.1
- net SCLK: now also IC101.36, R146.1; no longer IC103.36
- net VAP: now also C109.1, IC101.23, R140.2; no longer C110.1, IC103.23, R128.2
- net VBP: now also C110.1, IC101.22, R141.2; no longer C111.1, IC103.22, R129.2
- net VCC: now also C118.+, C122.1, C124.1, C125.2, IC101.26, R143.2, R145.2, R146.2, R147.2, R148.2, R149.2, R150.1; no longer C119.+, C121.1, C125.1, C126.2, IC103.26, R131.2, R132.2, R133.1
- net VCC_P: now also C126.2, C127.+, C128.1, IC103.3, R151.2, R152.2; no longer C127.2, C128.+, C130.1, IC105.3, R134.2, R135.2
- net VCP: now also C111.1, IC101.19, R142.2; no longer C112.1, IC103.19, R130.2
- net VN: now also C109.2, IC101.18, R137.1, R138.1, R139.1, X102.P$1; no longer C112.2, IC103.18, R122.1, R123.1, R124.1, X101.P$1
- net XTAL1: now also C116.2, IC101.27; no longer C104.2, IC103.27
- net XTAL2: now also C114.1, IC101.28; no longer C101.1, IC103.28
Routing:
- net VCC: track 108.6 -> 117.5 mm, vias 2 -> 3
- net SCLK: track 13.3 -> 19.4 mm
- net N$42: track 4.83 -> 0.00 mm
- net N$16: track 0.00 -> 4.83 mm
- net MISO: track 14.2 -> 18.7 mm
- net MOSI: track 20.1 -> 23.2 mm
- net !SS: track 16.4 -> 19.5 mm
- net GND: track 124.9 -> 127.8 mm, vias 6 -> 7
- net VCC_P: track 76.8 -> 77.9 mm
